File: IO-Board-2-X.brd (EAGLE design)
At the start: 160 x 100 mm, 209 parts, among them IC1 LP2950Z, IC2 LP2950Z, J1.1 TPPAD1-13, J1.2 TPPAD1-13, J1.3 TPPAD1-13, J1.4 TPPAD1-13, J1.5 TPPAD1-13, J1.6 TPPAD1-13, J1.7 TPPAD1-13, J1.8 TPPAD1-13, J2.1 TPPAD1-13, J2.2 TPPAD1-13, J2.3 TPPAD1-13, J2.4 TPPAD1-13, J2.5 TPPAD1-13, J2.6 TPPAD1-13, J2.7 TPPAD1-13, J2.8 TPPAD1-13, J3.1 TPPAD1-13, J3.2 TPPAD1-13, J3.3 TPPAD1-13, J3.4 TPPAD1-13, J3.5 TPPAD1-13, J3.6 TPPAD1-13, J3.7 TPPAD1-13, J3.8 TPPAD1-13, J4.5 TPPAD1-13, J4.6 TPPAD1-13, J4.7 TPPAD1-13, J4.8 TPPAD1-13, K1 FINDER-43.41, K2 FINDER-43.41, K3 FINDER-43.41, K4 FINDER-43.41, U1 ATTINY85V-10S, U2 ATTINY85V-10S

Commit message: IO-Board-2 Anpassung
Parts:
- added 433_RX, 433_TX, GPIO_24, J4.1, J4.2, J4.3, J4.4, PB0, PB1, PB2, PB3, PB4, PB5, PC3, PD0, PD1, PD2, PD3, PD4, PD5, PD6, PD7: TPPAD1-13, testpad:P1-13
- added C5, C7, C8: 100nF, rcl:C025-025X050
- added C6, C9: 10µF, rcl:E2-4
- added IC3: LM2936-5.0, LM2936:TO92-INLINE
- added JP1: (no value), jumper:JP2
- added JP2: (no value), jumper:JP4
- added Q1: 8MHz, crystal:HC49U-V
- added R13: 10k, rcl:0204/5
- C1: value 1µF -> 100nF
- C2: value 2,2µF -> 22pF
- C3: value 1µF -> 22pF
- C4: value 2,2µF -> 100nF
- IC1: value LP2950Z -> MEGA8-P; device linear:TO92 -> atmel:DIL28-3
- IC2: value LP2950Z -> LM2936-5.0; device linear:TO92 -> LM2936:TO92-INLINE
- R1, R2: device rcl:0204V -> rcl:0204/5
- R11, R6: value 1k5 -> 10k
- R12, R7: value 10k -> 1k5
- R3: device rcl:0204/5 -> rcl:0204V
- moved R3 108.0 mm to (20.3, 27.9), turned to 90 degrees
- moved IC1 106.1 mm to (36.8, 35.6), turned to 0 degrees
- moved C2 105.2 mm to (40.0, 22.9), turned to 0 degrees
- moved C1 99.5 mm to (36.8, 27.9), turned to 180 degrees
- moved C3 60.5 mm to (41.3, 25.4), turned to 0 degrees
- moved L 57.5 mm to (152.4, 76.2), turned to 270 degrees
- moved L1 57.5 mm to (152.4, 50.8), turned to 270 degrees
- moved L_RAUS 56.6 mm to (152.4, 96.5), turned to 270 degrees
- moved L_RAUS1 56.6 mm to (152.4, 71.1), turned to 270 degrees
- moved J5 55.9 mm to (97.8, 86.4), turned to 270 degrees
- moved J6 55.9 mm to (97.8, 61.0), turned to 270 degrees
- moved L_REIN 53.7 mm to (152.4, 83.8), turned to 270 degrees
- moved L_REIN1 53.7 mm to (152.4, 58.4), turned to 270 degrees
- moved R8 44.2 mm to (135.9, 36.2)
- moved R1 41.5 mm to (47.0, 49.5)
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Connections:
- removed net GND.2: R2.1, SV1.29, SV1.29T
- new net +5V_2: JP1.2, JP2.1, SV1.28, SV1.28T
- new net 433MHZ_INT: IC1.25, SV1.27, SV1.27T
- new net GND_2: JP1.3, JP2.4, R2.1, SV1.29, SV1.29T
- new net N$1: J4.4, J4.4.TP
- new net N$14: IC1.11, PD5.TP
- new net N$16: IC1.13, PD7.TP
- new net N$17: IC1.14, PB0.TP
- new net N$18: IC1.15, PB1.TP
- new net N$19: IC1.16, PB2.TP
- new net N$20: IC1.17, PB3.TP
- new net N$21: IC1.18, PB4.TP
- new net N$22: IC1.19, PB5.TP
- new net N$23: C3.2, IC1.10, Q1.1
- new net N$24: C2.2, IC1.9, Q1.2
- new net N$25: MOSI.TP, R4.2, S1.3, S1.4, U1.5
- new net N$26: MISO.TP, R5.2, S2.3, S2.4, U1.6
- new net N$27: R6.2, S3.3, S3.4, SCK.TP, U1.7
- new net N$28: R7.1, U1.3
- new net N$29: LED1.A, R7.2
- new net N$31: R8.1, RESET.TP, U1.1
- new net N$32: MOSI1.TP, R9.2, S4.3, S4.4, U2.5
- new net N$33: MISO1.TP, R10.2, S5.3, S5.4, U2.6
- new net N$34: R11.2, S6.3, S6.4, SCK1.TP, U2.7
- new net N$35: R12.1, U2.3
- new net N$52: LED2.A, R12.2
- new net N$54: R13.1, RESET1.TP, U2.1
- net +12V: now also C4.1, IC2.VIN; no longer C1.1, IC1.3
- net +12V1: now also C7.1, IC3.VIN; no longer C3.1, IC2.3
- net +3V3: now also C1.2, IC1.20, IC1.21, IC1.7, R3.1
- net +5V: no longer J4.1
- net +5V1: now also C5.1, C6.+, IC2.VO, R6.1, R8.2; no longer C2.1, IC1.1, R3.1, R7.2
- net +5V2: now also C8.1, C9.+, IC3.VO, R11.1, R13.2; no longer C4.1, IC2.1, R12.2, R8.1
- net 433MHZ_RX: now also 433_RX.TP, JP2.2; no longer J4.4
- net 433MHZ_TX: now also 433_TX.TP, IC1.24, JP1.1; no longer J4.3, SV1.27, SV1.27T
- net GND: now also C1.1, C2.1, C3.1, IC1.22, IC1.8; no longer J4.2
- net GND1: now also C4.2, C5.2, C6.-, IC2.GND; no longer C1.2, C2.2, IC1.2
- net GND2: now also C7.2, C8.2, C9.-, IC3.GND; no longer C3.2, C4.2, IC2.2
- net N$10: now also IC1.3, PD1.TP; no longer MISO1.TP, R9.2, S5.3, S5.4, U2.6
- net N$11: now also IC1.4, PD2.TP; no longer R10.2, S6.3, S6.4, SCK1.TP, U2.7
- net N$12: now also IC1.5, PD3.TP; no longer R11.1, U2.3
- net N$13: now also IC1.6, PD4.TP; no longer LED2.A, R11.2
- net N$15: now also IC1.12, PD6.TP; no longer R12.1, RESET1.TP, U2.1
- net N$2: now also IC1.23; no longer SV1.26, SV1.26T
- net N$3: now also J4.3, J4.3.TP; no longer MOSI.TP, R3.2, S1.3, S1.4, U1.5
- net N$4: now also J4.2, J4.2.TP; no longer MISO.TP, R4.2, S2.3, S2.4, U1.6
- net N$5: now also J4.1, J4.1.TP; no longer R5.2, S3.3, S3.4, SCK.TP, U1.7
- net N$6: now also IC1.1, R3.2; no longer R6.1, U1.3
- net N$7: now also GPIO_24.TP, SV1.26, SV1.26T; no longer LED1.A, R6.2
- net N$8: now also IC1.26, PC3.TP; no longer R7.1, RESET.TP, U1.1
- net N$9: now also IC1.2, PD0.TP; no longer MOSI1.TP, R8.2, S4.3, S4.4, U2.5
- net SCL: now also IC1.28
- net SDA: now also IC1.27
Routing:
- net 433MHZ_TX: track 124.9 -> 16.3 mm
- net 433MHZ_RX: track 108.8 -> 6.35 mm
- net GND_2: track 0.00 -> 90.1 mm
- net +5V_2: track 0.00 -> 77.4 mm
- net 433MHZ_INT: track 0.00 -> 59.0 mm
- net +3V3: track 24.9 -> 82.3 mm
- net +5V: track 67.4 -> 25.8 mm
- net N$34: track 0.00 -> 40.5 mm
- net N$27: track 0.00 -> 40.5 mm
- net N$11: track 40.5 -> 3.81 mm
- net N$26: track 0.00 -> 35.1 mm
- net N$33: track 0.00 -> 35.1 mm
- net SDA: track 0.00 -> 34.3 mm
- net N$25: track 0.00 -> 33.9 mm
- net N$32: track 0.00 -> 33.9 mm
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- added copper zone on layer 16, net GND
- removed copper zone on layer 16, net GND1
- removed copper zone on layer 16, net GND2
Other:
- outline, holes or cut-outs redrawn
- board text added: "+"
- board text added: "-"
- board text added: "24"
- board text added: "433MHz Handsender Rev 2016/08 (c) Peter Müller"
- board text added: "433MHz RX"
- board text added: "433MHz TX"
- board text added: "Bitte hier schneiden"
- board text added: "HomePi IO-Board #2 Rev 2016/08 (c) Peter Müller"
- board text removed: "433MHz Handsender Rev 2016/07 (c) Peter Müller"
- board text removed: "HomePi IO-Board Rev 2016/07 (c) Peter Müller"
