File: Pi.sch (EAGLE design)
At the start: 14 parts, among them IC1 DS18B20, X1 RASPI_GPIO_B+#_PIN, X2 HDD, 5V 700mA, X3 MAC64L

Commit message: Platinen angepasst, Backplane
Connections:
- net +5V_INT: now also X2-1.1; no longer C1.+, X1.5V0A, X1.5V0B
- net +5V_INT2: now also C1.+, X1.5V0A, X1.5V0B; no longer X2-1.1
Changed lines of the file:
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@@
 <net name="+5V_INT2" class="0">
-<segment>
-<pinref part="X2" gate="-1" pin="1"/>
-<wire x1="137.16" y1="152.4" x2="144.78" y2="152.4" width="0.1524" layer="91"/>
-<label x="137.16" y="152.4" size="1.778" layer="95" rot="MR0"/>
-</segment>
 <segment>
 <pinref part="X3" gate="G$1" pin="A28"/>
@@
 <label x="66.04" y="96.52" size="1.778" layer="95"/>
 </segment>
-</net>
-<net name="+5V_INT" class="0">
 <segment>
 <pinref part="X1" gate="G$1" pin="5V0A"/>
@@
 <junction x="187.96" y="149.86"/>
 </segment>
+</net>
+<net name="+5V_INT" class="0">
 <segment>
 <pinref part="X3" gate="G$1" pin="A1"/>
@@
 <label x="66.04" y="165.1" size="1.778" layer="95"/>
 </segment>
+<segment>
+<pinref part="X2" gate="-1" pin="1"/>
+<wire x1="137.16" y1="152.4" x2="144.78" y2="152.4" width="0.1524" layer="91"/>
+<label x="137.16" y="152.4" size="1.778" layer="95" rot="MR0"/>
+</segment>
 </net>
