File: Backplane-2.brd (EAGLE design)
At the start: 97.8 x 84 mm, 6 parts, among them X1 FAC64S, X2 FAC64S, X3 FAC64S, X4 FAC64S

Commit message: Layouts angepasst
Connections:
- net A26 renamed A25
Other:
- board text added: "HomePi Backplane"
- board text added: "Rev 2019/04 (c) Peter Müller"
Changed lines of the file:
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@@
 <dimension x1="16.51" y1="41.91" x2="-3.81" y2="41.91" x3="6.35" y3="-11.43" textsize="1.778" layer="47"/>
 <dimension x1="82.55" y1="41.91" x2="97.79" y2="41.91" x3="90.17" y3="-11.43" textsize="1.778" layer="47"/>
+<text x="30.48" y="63.5" size="2.54" layer="25" font="vector" ratio="15" rot="SR270" align="center">HomePi
+Backplane</text>
+<text x="30.48" y="21.59" size="2.54" layer="25" font="vector" ratio="15" rot="SR270" align="center">Rev 2019/04
+(c) Peter Müller</text>
 </plain>
 <attributes>
@@
 <class number="0" name="default" width="0" drill="0">
 </class>
+<class number="1" name="24V" width="0.8128" drill="0">
+<clearance class="1" value="0.4064"/>
+</class>
 </classes>
-<designrules name="platinenbelichter">
+<designrules name="allpcb">
 <description language="de">&lt;b&gt;EAGLE Design Rules&lt;/b&gt;
 &lt;p&gt;
@@
 <param name="mtCopper" value="0.035mm 0.035mm 0.035mm 0.035mm 0.035mm 0.035mm 0.035mm 0.035mm 0.035mm 0.035mm 0.035mm 0.035mm 0.035mm 0.035mm 0.035mm 0.035mm"/>
 <param name="mtIsolate" value="1.5mm 0.15mm 0.2mm 0.15mm 0.2mm 0.15mm 0.2mm 0.15mm 0.2mm 0.15mm 0.2mm 0.15mm 0.2mm 0.15mm 0.2mm"/>
-<param name="mdWireWire" value="10mil"/>
-<param name="mdWirePad" value="10mil"/>
-<param name="mdWireVia" value="10mil"/>
-<param name="mdPadPad" value="10mil"/>
-<param name="mdPadVia" value="10mil"/>
-<param name="mdViaVia" value="10mil"/>
-<param name="mdSmdPad" value="10mil"/>
-<param name="mdSmdVia" value="10mil"/>
-<param name="mdSmdSmd" value="10mil"/>
+<param name="mdWireWire" value="6mil"/>
+<param name="mdWirePad" value="6mil"/>
+<param name="mdWireVia" value="6mil"/>
+<param name="mdPadPad" value="6mil"/>
+<param name="mdPadVia" value="6mil"/>
+<param name="mdViaVia" value="6mil"/>
+<param name="mdSmdPad" value="6mil"/>
+<param name="mdSmdVia" value="6mil"/>
+<param name="mdSmdSmd" value="6mil"/>
 <param name="mdViaViaSameLayer" value="8mil"/>
 <param name="mnLayersViaInSmd" value="2"/>
@@
 <param name="mdDrill" value="8mil"/>
 <param name="mdSmdStop" value="0mil"/>
-<param name="msWidth" value="10mil"/>
-<param name="msDrill" value="24mil"/>
+<param name="msWidth" value="4mil"/>
+<param name="msDrill" value="0.3mm"/>
 <param name="msMicroVia" value="9.99mm"/>
 <param name="msBlindViaRatio" value="0.5"/>
@@
 <wire x1="87.63" y1="17.78" x2="90.805" y2="17.78" width="0.4064" layer="1"/>
 </signal>
-<signal name="+24V">
+<signal name="+24V" class="1">
 <contactref element="X1" pad="C32"/>
 <contactref element="X1" pad="A32"/>
@@
 <wire x1="87.63" y1="22.86" x2="90.805" y2="22.86" width="0.4064" layer="1"/>
 </signal>
-<signal name="A26">
+<signal name="A25">
 <contactref element="X1" pad="A25"/>
 <contactref element="X2" pad="A25"/>
@@
 </board>
 </drawing>
+<compatibility>
+<note version="6.3" minversion="6.2.2" severity="warning">
+Since Version 6.2.2 text objects can contain more than one line,
+which will not be processed correctly with this version.
+</note>
+</compatibility>
 </eagle>

Commit message: Layouts angepasst
Parts:
- X1, X2, X3, X4: value FAC64S -> FAC64SNO_DRILL; device con-vg:FAC64S -> my-con-vg:FAC64S_NO_DRILL
Changed lines of the file:
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@@
 <layer number="42" name="bRestrict" color="1" fill="10" visible="yes" active="yes"/>
 <layer number="43" name="vRestrict" color="2" fill="10" visible="yes" active="yes"/>
-<layer number="44" name="Drills" color="7" fill="1" visible="no" active="yes"/>
-<layer number="45" name="Holes" color="7" fill="1" visible="no" active="yes"/>
-<layer number="46" name="Milling" color="3" fill="1" visible="no" active="yes"/>
+<layer number="44" name="Drills" color="7" fill="1" visible="yes" active="yes"/>
+<layer number="45" name="Holes" color="7" fill="1" visible="yes" active="yes"/>
+<layer number="46" name="Milling" color="3" fill="1" visible="yes" active="yes"/>
 <layer number="47" name="Measures" color="7" fill="1" visible="yes" active="yes"/>
 <layer number="48" name="Document" color="7" fill="1" visible="yes" active="yes"/>
@@
 <board>
 <plain>
-<wire x1="0" y1="0" x2="97.79" y2="0" width="0.2" layer="20"/>
-<wire x1="97.79" y1="0" x2="97.79" y2="84" width="0.2" layer="20"/>
-<wire x1="97.79" y1="84" x2="0" y2="84" width="0.2" layer="20"/>
-<wire x1="0" y1="84" x2="0" y2="0" width="0.2" layer="20"/>
+<wire x1="0" y1="0" x2="97.79" y2="0" width="0.254" layer="20"/>
+<wire x1="97.79" y1="0" x2="97.79" y2="84" width="0.254" layer="20"/>
+<wire x1="97.79" y1="84" x2="0" y2="84" width="0.254" layer="20"/>
+<wire x1="0" y1="84" x2="0" y2="0" width="0.254" layer="20"/>
 <dimension x1="16.51" y1="41.91" x2="41.91" y2="41.91" x3="29.21" y3="-11.43" textsize="1.778" layer="47" visible="yes"/>
 <dimension x1="41.91" y1="41.91" x2="62.23" y2="41.91" x3="52.07" y3="-11.43" textsize="1.778" layer="47" visible="yes"/>
@@
 </autorouter>
 <elements>
-<element name="X1" library="con-vg" package="FAC64S" value="FAC64S" x="16.51" y="41.91" smashed="yes">
+<element name="X1" library="my-con-vg" package="FAC64S_NO_DRILL" value="FAC64SNO_DRILL" x="16.51" y="41.91" smashed="yes">
 <attribute name="NAME" x="22.479" y="0.2" size="1.27" layer="25" ratio="10" rot="SR0"/>
 <attribute name="VALUE" x="8.128" y="5.08" size="1.27" layer="27" ratio="10" rot="R90"/>
 </element>
-<element name="X2" library="con-vg" package="FAC64S" value="FAC64S" x="41.91" y="41.91" smashed="yes">
+<element name="X2" library="my-con-vg" package="FAC64S_NO_DRILL" value="FAC64SNO_DRILL" x="41.91" y="41.91" smashed="yes">
 <attribute name="NAME" x="47.879" y="0.2" size="1.27" layer="25" ratio="10" rot="SR0"/>
 <attribute name="VALUE" x="36.068" y="5.08" size="1.27" layer="27" ratio="10" rot="R90"/>
 </element>
-<element name="X3" library="con-vg" package="FAC64S" value="FAC64S" x="62.23" y="41.91" smashed="yes">
+<element name="X3" library="my-con-vg" package="FAC64S_NO_DRILL" value="FAC64SNO_DRILL" x="62.23" y="41.91" smashed="yes">
 <attribute name="NAME" x="68.199" y="0.2" size="1.27" layer="25" ratio="10" rot="SR0"/>
 <attribute name="VALUE" x="56.388" y="5.08" size="1.27" layer="27" ratio="10" rot="R90"/>
 </element>
-<element name="X4" library="con-vg" package="FAC64S" value="FAC64S" x="82.55" y="41.91" smashed="yes">
+<element name="X4" library="my-con-vg" package="FAC64S_NO_DRILL" value="FAC64SNO_DRILL" x="82.55" y="41.91" smashed="yes">
 <attribute name="NAME" x="88.519" y="0.2" size="1.27" layer="25" ratio="10" rot="SR0"/>
 <attribute name="VALUE" x="76.708" y="5.08" size="1.27" layer="27" ratio="10" rot="R90"/>
