File: Backplane-2.sch (EAGLE design)
At the start: 6 parts, among them X1 FAC64S, X2 FAC64S, X3 FAC64S, X4 FAC64S

Commit message: Layouts angepasst
Connections:
- net A26 renamed A25
Changed lines of the file:
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@@
 <class number="0" name="default" width="0" drill="0">
+</class>
+<class number="1" name="24V" width="0.8128" drill="0">
+<clearance class="1" value="0.4064"/>
 </class>
 </classes>
@@
 </segment>
 </net>
-<net name="+24V" class="0">
+<net name="+24V" class="1">
 <segment>
 <pinref part="X1" gate="G$1" pin="C32"/>
@@
 </segment>
 </net>
-<net name="A26" class="0">
+<net name="A25" class="0">
 <segment>
 <pinref part="X1" gate="G$1" pin="A25"/>
@@
 </segment>
 </net>
-<net name="+24V" class="0">
+<net name="+24V" class="1">
 <segment>
 <wire x1="162.56" y1="60.96" x2="157.48" y2="60.96" width="0.1524" layer="91"/>
@@
 </segment>
 </net>
-<net name="A26" class="0">
+<net name="A25" class="0">
 <segment>
 <wire x1="162.56" y1="78.74" x2="157.48" y2="78.74" width="0.1524" layer="91"/>

Commit message: Layouts angepasst
Parts:
- X1, X2, X3, X4: value FAC64S -> FAC64SNO_DRILL; device con-vg:FAC64S -> my-con-vg:FAC64SNO_DRILL
Changed lines of the file:
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@@
 <parts>
 <part name="FRAME1" library="frames" deviceset="A4L-LOC" device=""/>
-<part name="X1" library="con-vg" deviceset="FAC64S" device=""/>
-<part name="X2" library="con-vg" deviceset="FAC64S" device=""/>
-<part name="X3" library="con-vg" deviceset="FAC64S" device=""/>
-<part name="X4" library="con-vg" deviceset="FAC64S" device=""/>
+<part name="X1" library="my-con-vg" deviceset="FAC64S" device="NO_DRILL"/>
+<part name="X2" library="my-con-vg" deviceset="FAC64S" device="NO_DRILL"/>
+<part name="X3" library="my-con-vg" deviceset="FAC64S" device="NO_DRILL"/>
+<part name="X4" library="my-con-vg" deviceset="FAC64S" device="NO_DRILL"/>
 <part name="FRAME2" library="frames" deviceset="A4L-LOC" device=""/>
 <part name="SV1" library="64-pol-verbinder" deviceset="FE32-2W" device=""/>
