File: Pi-4.brd (EAGLE design)
At the start: 140 x 100 mm, 15 parts, among them IC1 DS18B20, X1 RASPI_GPIO_B+#_PIN, X2 HDD, 5V 700mA, X3 MAC64L

Commit message: Layouts angepasst
Parts:
- moved R3 49.5 mm to (92.1, 61.6), flipped to the bottom, turned to 180 degrees
- moved X2 39.4 mm to (96.5, 8.89)
- moved R1 38.8 mm to (92.1, 19.7)
- moved R2 38.8 mm to (92.1, 24.8)
- moved LED1 38.8 mm to (97.2, 18.4)
- moved LED2 38.8 mm to (97.2, 23.5)
- moved OK1 37.4 mm to (94.0, 70.5), flipped to the bottom, turned to 0 degrees
- moved JP2 21.1 mm to (95.9, 87.6)
- moved C1 21.0 mm to (31.1, 92.5)
- moved X1 21.0 mm to (66.7, 90.2)
- moved RPI1 21.0 mm to (34.3, 29.8)
- moved IC1 15.2 mm to (22.9, 20.3)
- moved R4 15.2 mm to (26.0, 25.4)
- moved U$1 0.90 mm to (15.9, 8.89)
Routing:
- net +5V_INT: track 156.9 -> 102.3 mm
- net +3,3V: track 159.2 -> 105.8 mm, vias 0 -> 1
- net GPIO.27: track 135.7 -> 112.2 mm
- net GPIO.26: track 106.9 -> 84.0 mm
- net GPIO.17: track 86.6 -> 65.5 mm
- net GPIO.18: track 86.6 -> 65.8 mm
- net GPIO.23: track 86.1 -> 65.3 mm
- net GPIO.24: track 88.3 -> 67.5 mm
- net GPIO.22: track 85.7 -> 64.9 mm
- net +5V_INT2: track 65.7 -> 45.3 mm
- net GPIO.21: track 122.1 -> 101.9 mm
- net SPI_CE1: track 115.4 -> 95.7 mm
- net GPIO.25: track 92.0 -> 72.3 mm
- net SPI_CE0: track 118.2 -> 98.5 mm
- net GPIO.20: track 119.4 -> 99.7 mm
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Other:
- board size 140 x 100 mm -> 100 x 100 mm
- board text added: "Pi- Reset"
- board text removed: "Pi-Reset"
