File: Stromversorgung-2.brd (EAGLE design)
At the start: 80 x 100 mm, 16 parts, among them J1 DCJ0202, U1 TSR 2-2450, U2 TSR 1-2433, U3 TSR 2-2450, X1 Ein/Aus, X2 MAC64L

Commit message: Layouts angepasst
Parts:
- R1, R2, R3, R4: device rcl:0204/5 -> rcl:R1206
- U1, U3: value TSR 2-2450 -> TSR2-2450; device _traco_tsr-1:TSR-1 -> TSR:TSR2
- U2: value TSR 1-2433 -> TSR1-2433; device _traco_tsr-1:TSR-1 -> TSR:TSR1
- X1: device con-phoenix-508:MSTBV2 -> con-phoenix-508:MSTBA2
- moved LED4 29.1 mm to (33.7, 33.7), turned to 90 degrees
- moved LED1 28.8 mm to (33.7, 47.6), turned to 90 degrees
- moved LED2 28.6 mm to (33.7, 64.8), turned to 90 degrees
- moved LED3 28.6 mm to (33.7, 81.9), turned to 90 degrees
- moved R4 28.5 mm to (28.6, 32.4)
- moved R1 25.4 mm to (28.6, 46.4)
- moved R2 25.2 mm to (28.6, 63.5)
- moved R3 25.0 mm to (28.6, 80.6)
- moved X1 21.7 mm to (36.8, 23.5), turned to 90 degrees
- moved J1 20.4 mm to (31.1, 10.2)
- moved C1 17.7 mm to (29.8, 40.3), turned to 270 degrees
- moved U1 17.5 mm to (21.6, 43.8)
- moved U2 17.1 mm to (21.6, 61.0)
- moved U3 16.8 mm to (21.6, 78.1)
- moved C2 16.7 mm to (29.8, 74.6), turned to 270 degrees
Connections:
- net +24V: now also X1.2; no longer X1.1
- net GND: now also X2.A11, X2.A13, X2.A27, X2.C13
- net N$1: now also X1.1; no longer X1.2
Routing:
- net +5V_INT: track 146.6 -> 98.0 mm
- net +3,3V: track 102.5 -> 71.8 mm, vias 0 -> 1
- net +5V_EXT: track 46.8 -> 24.4 mm
- net +24V: track 157.5 -> 149.3 mm
- net N$1: track 18.9 -> 14.9 mm
- net N$8: track 6.35 -> 3.66 mm
- net N$7: track 6.35 -> 3.66 mm
- net N$6: track 6.35 -> 3.66 mm
Other:
- board size 80 x 100 mm -> 40.6 x 100 mm
- board text added: "+5V"
- board text added: "HomePi Spannungsversorgung"
- board text added: "Rev 2019/04 (c) Peter Müller"
- board text removed: "+5V int."
- board text removed: "HomePi Stromversorgung Rev 2019/04 (c) Peter Müller"

Commit message: Layouts angepasst
Parts:
- removed J1: DCJ0202, con-jack:DCJ0202
- added X3: Ein/Aus, con-phoenix-508:MSTBA2
- U3: value TSR2-2450 -> TSR1-2425; device TSR:TSR2 -> TSR:TSR1
Connections:
- removed net N$1: J1.1, X1.1
- new net +24V_IN: X1.1, X3.2
- net GND: now also X3.1; no longer J1.3
Routing:
- net N$1: track 14.9 -> 0.00 mm
- net +24V_IN: track 0.00 -> 11.8 mm
- net +24V: track 149.3 -> 147.6 mm
Other:
- board text added: "+"
- board text added: "-"
Changed lines of the file:
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@@
 <setting verticaltext="up"/>
 </settings>
-<grid distance="25" unitdist="mil" unit="mm" style="lines" multiple="1" display="no" altdistance="12.5" altunitdist="mil" altunit="mil"/>
+<grid distance="25" unitdist="mil" unit="mm" style="lines" multiple="1" display="yes" altdistance="12.5" altunitdist="mil" altunit="mil"/>
 <layers>
 <layer number="1" name="Top" color="4" fill="1" visible="yes" active="yes"/>
@@
 <text x="11.7475" y="67.31" size="1.9304" layer="25" font="vector" ratio="15" rot="R90" align="top-center">Rev 2019/04
 (c) Peter Müller</text>
+<text x="28.575" y="12.7" size="2.54" layer="25" font="vector" ratio="15" rot="R90" align="center">+</text>
+<text x="28.575" y="7.62" size="2.54" layer="25" font="vector" ratio="15" rot="R90" align="center">-</text>
 </plain>
 <attributes>
@@
 <element name="U1" library="TSR" package="TSR2" value="TSR2-2450" x="21.59" y="43.815" smashed="yes" rot="R90"/>
 <element name="U2" library="TSR" package="TSR1" value="TSR1-2433" x="21.59" y="60.96" smashed="yes" rot="R90"/>
-<element name="U3" library="TSR" package="TSR2" value="TSR2-2450" x="21.59" y="78.105" smashed="yes" rot="R90"/>
-<element name="J1" library="con-jack" package="DCJ0202" value="DCJ0202" x="31.115" y="10.16" smashed="yes" rot="R90">
-<attribute name="OC_FARNELL" value="unknown" x="31.115" y="10.16" size="1.778" layer="27" rot="R90" display="off"/>
-<attribute name="MPN" value="" x="31.115" y="10.16" size="1.778" layer="27" rot="R90" display="off"/>
-<attribute name="OC_NEWARK" value="unknown" x="31.115" y="10.16" size="1.778" layer="27" rot="R90" display="off"/>
-<attribute name="MF" value="" x="31.115" y="10.16" size="1.778" layer="27" rot="R90" display="off"/>
-<attribute name="VALUE" x="41.275" y="5.08" size="1.27" layer="27" rot="R180"/>
-</element>
+<element name="U3" library="TSR" package="TSR1" value="TSR1-2425" x="21.59" y="78.105" smashed="yes" rot="R90"/>
 <element name="X2" library="con-vg" package="MAC64L" value="MAC64L" x="2.54" y="49.53" locked="yes" smashed="yes" rot="R180">
 <attribute name="VALUE" x="-5.08" y="60.9854" size="1.27" layer="27" ratio="10" rot="R270"/>
@@
 <element name="LED4" library="led" package="LED3MM" value="2mA ge" x="33.655" y="33.655" smashed="yes" rot="R90">
 <attribute name="VALUE" x="35.306" y="35.56" size="1.27" layer="27" ratio="10" rot="R90"/>
+</element>
+<element name="X3" library="con-phoenix-508" package="MSTBA2" value="Ein/Aus" x="36.83" y="10.16" smashed="yes" rot="R90">
+<attribute name="MPN" value="1757242" x="36.83" y="10.16" size="1.778" layer="27" ratio="15" rot="R90" display="off"/>
+<attribute name="OC_FARNELL" value="3705171" x="36.83" y="10.16" size="1.778" layer="27" ratio="15" rot="R90" display="off"/>
+<attribute name="MF" value="FARNELL" x="36.83" y="10.16" size="1.778" layer="27" ratio="15" rot="R90" display="off"/>
+<attribute name="OC_NEWARK" value="71C4161" x="36.83" y="10.16" size="1.778" layer="27" ratio="15" rot="R90" display="off"/>
+<attribute name="VALUE" x="36.83" y="5.08" size="1.778" layer="27" ratio="10" rot="R90"/>
 </element>
 </elements>
@@
 <contactref element="X2" pad="C31"/>
 <wire x1="10.16" y1="86.36" x2="5.08" y2="86.36" width="1.27" layer="1"/>
-<wire x1="21.59" y1="80.645" x2="27.153" y2="80.645" width="0.4064" layer="1"/>
-<wire x1="21.59" y1="80.645" x2="18.415" y2="80.645" width="1.27" layer="1"/>
+<wire x1="23.34" y1="80.645" x2="27.153" y2="80.645" width="0.4064" layer="1"/>
+<wire x1="23.34" y1="80.645" x2="18.415" y2="80.645" width="1.27" layer="1"/>
 <wire x1="18.415" y1="80.645" x2="12.7" y2="86.36" width="1.27" layer="1"/>
 <wire x1="12.7" y1="86.36" x2="10.16" y2="86.36" width="1.27" layer="1"/>
@@
 <wire x1="28.575" y1="26.035" x2="31.75" y2="26.035" width="0.4064" layer="1"/>
 <wire x1="36.83" y1="83.82" x2="31.75" y2="88.9" width="1.27" layer="1"/>
-<wire x1="21.59" y1="75.565" x2="29.841" y2="75.565" width="1.27" layer="1"/>
+<wire x1="23.34" y1="75.565" x2="29.841" y2="75.565" width="1.27" layer="1"/>
 <wire x1="29.841" y1="75.565" x2="29.845" y2="75.569" width="1.27" layer="1"/>
 <wire x1="29.845" y1="75.569" x2="36.826" y2="75.569" width="1.27" layer="1"/>
@@
 <contactref element="LED2" pad="K"/>
 <contactref element="LED3" pad="K"/>
-<contactref element="J1" pad="3"/>
 <contactref element="X2" pad="A29"/>
 <contactref element="X2" pad="A30"/>
@@
 <contactref element="X2" pad="C13"/>
 <contactref element="X2" pad="A27"/>
+<contactref element="X3" pad="1"/>
 </signal>
 <signal name="N$3">
@@
 <contactref element="X2" pad="A7"/>
 </signal>
-<signal name="N$1">
-<contactref element="J1" pad="1"/>
+<signal name="+24V_IN">
+<contactref element="X3" pad="2"/>
 <contactref element="X1" pad="1"/>
-<wire x1="28.015" y1="10.16" x2="28.015" y2="12.625" width="1.27" layer="1"/>
-<wire x1="28.015" y1="12.625" x2="26.67" y2="13.97" width="1.27" layer="1"/>
-<wire x1="26.67" y1="13.97" x2="26.67" y2="18.415" width="1.27" layer="1"/>
-<wire x1="26.67" y1="18.415" x2="29.21" y2="20.955" width="1.27" layer="1"/>
-<wire x1="29.21" y1="20.955" x2="31.75" y2="20.955" width="1.27" layer="1"/>
+<wire x1="31.75" y1="20.955" x2="30.48" y2="20.955" width="1.27" layer="1"/>
+<wire x1="30.48" y1="20.955" x2="29.21" y2="19.685" width="1.27" layer="1"/>
+<wire x1="29.21" y1="19.685" x2="29.21" y2="13.97" width="1.27" layer="1"/>
+<wire x1="29.21" y1="13.97" x2="30.48" y2="12.7" width="1.27" layer="1"/>
+<wire x1="30.48" y1="12.7" x2="31.75" y2="12.7" width="1.27" layer="1"/>
 </signal>
 </signals>

Commit message: Layouts angepasst
Parts:
- added D1: MBRS 540T3G, diode:SMC
- added F1: 30V / 2,5A, fuse:LITTLEFUSE
- added U$1: (no value), cryCode-Logo:30MM
- X3: value Ein/Aus -> Eingang
- moved X1 10.2 mm to (47.0, 24.8)
- moved X3 10.2 mm to (47.0, 9.53)
- moved R4 10.2 mm to (38.7, 33.0)
- moved LED4 10.2 mm to (43.8, 34.3)
- moved R1 10.2 mm to (38.7, 46.4)
- moved R2 10.2 mm to (38.7, 63.5)
- moved R3 10.2 mm to (38.7, 80.6)
- moved LED1 10.2 mm to (43.8, 47.6)
- moved LED2 10.2 mm to (43.8, 64.8)
- moved LED3 10.2 mm to (43.8, 81.9)
- moved C1 4.45 mm to (34.3, 40.3)
- moved C2 4.45 mm to (34.3, 74.6)
- moved U1 4.45 mm to (26.0, 43.8)
- moved U2 4.45 mm to (26.0, 61.0)
- moved U3 4.45 mm to (26.0, 78.1)
Connections:
- new net +24V_IN_RAW: F1.2, X3.2
- net +24V: now also D1.C
- net +24V_IN: now also F1.1; no longer X3.2
- net GND: now also D1.A
Routing:
- net +24V: track 147.6 -> 281.4 mm
- net +5V_EXT: track 24.4 -> 34.6 mm
- net +3,3V: track 71.8 -> 81.9 mm
- net +5V_INT: track 98.0 -> 107.9 mm
- net +24V_IN_RAW: track 0.00 -> 8.89 mm
- net +24V_IN: track 11.8 -> 8.89 mm
- added copper zone on layer 1, net TOP
Other:
- board size 40.6 x 100 mm -> 52.1 x 100 mm
- board text added: "BOT"
- board text added: "Rev 2019/05 (c) Peter Müller"
- board text added: "TOP"
- board text removed: "Rev 2019/04 (c) Peter Müller"
