File: Platinen-Adapter.sch (EAGLE design)
At the start: 2 parts, among them X1 MAC64L

Commit message: Beschriftung hinzugefügt
Other:
- note added: "HomePi - Platinenadapter Rev. 2019/05"
Changed lines of the file:
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@@
 <sheet>
 <plain>
+<text x="160.02" y="15.24" size="2.54" layer="94" align="top-left">HomePi - Platinenadapter
+Rev. 2019/05</text>
 </plain>
 <instances>
@@
 </schematic>
 </drawing>
+<compatibility>
+<note version="6.3" minversion="6.2.2" severity="warning">
+Since Version 6.2.2 text objects can contain more than one line,
+which will not be processed correctly with this version.
+</note>
+</compatibility>
 </eagle>
