File: CAN-Shield.sch (EAGLE design)
At the start: 28 parts, among them IC1 LM2937IMP-5.0, IC2 MEGA8-AI, IC3 MCP2515T-I/SO, Q1 EUROQUARTZ-MMJ, Q2 EUROQUARTZ-MMJ, Q3 BC847ASMD, Q4 BC847ASMD, U1 MCP2562-E/SN

Commit message: CAN-Schield hinzugefügt, CanBus-UP-Schalter fertiggestellt
Parts:
- removed C10, C11: (no value), rcl:C-EUC0805
- removed C6: 22pF, rcl:C-EUC0805
- removed C7, C8, C9: 100nF, rcl:C-EUC0805
- removed IC3: MCP2515T-I/SO, mcp2515_2551_2562:MCP2515T-I/SO
- removed ISP1: ISPVIAS-ONLY-1.27MM, pogo-isp:ISPVIAS-ONLY-1.27MM
- removed LSP1, LSP2: LSP13, solpad:LSP13
- removed Q2: EUROQUARTZ-MMJ, crystal-smd:EUROQUARTZ-MMJ
- removed Q3, Q4: BC847ASMD, transistor-npn:BC847ASMD
- removed R3, R4: 4k7, rcl:R-EU_R0805
- removed RN1: (no value), resistor-dil:4R-N0603-ARC
- removed SV1: (no value), con-lstb:MA06-1
- removed U1: MCP2562-E/SN, mcp2515_2551_2562:MCP2562-E/SN
- added J1: (no value), can-bus:RJ45-CAN
- added JP1: (no value), jumper:JP1E
- added JP2: (no value), jumper:JP2E
- added X1: RASPI_GPIO_B+#_PIN, raspberrypi_bastelstube_v13:RASPI_GPIO_B+#_PIN
- added X2: (no value), pinhead:PINHD-1X7
- added X3: (no value), pinhead:PINHD-1X4
- C1, C2: value (none) -> 100nF; device rcl:C-EUC0805 -> rcl:C-EUC1206
- C3: value 22pF -> 100nF; device rcl:C-EUC0805 -> rcl:C-EUC1206
- C4, C5: device rcl:C-EUC0805 -> rcl:C-EUC1206
- IC1: value LM2937IMP-5.0 -> MCP2515-I/SO; device lm2937:LM2937IMP-5.0 -> mcp2515_2551_2562:MCP2515-I/SO
- IC2: value MEGA8-AI -> MCP2562-E/SN; device atmel:MEGA8-AI -> mcp2515_2551_2562:MCP2562-E/SN
- Q1: value EUROQUARTZ-MMJ -> 16MHz; device crystal-smd:EUROQUARTZ-MMJ -> crystal:CRYSTALHC49UP
- R1: value 10k -> 4k7; device rcl:R-EU_R0805 -> rcl:R-EU_R1206
- R2: value 4k7 -> 120R; device rcl:R-EU_R0805 -> rcl:R-EU_R1206
Connections:
- removed net CS: IC2.PB2(SS/OC1B), IC3.CS
- removed net IN1: C11.1, IC2.PC2(ADC2), RN1D.2
- removed net IN2: C10.1, IC2.PC3(ADC3), RN1A.2
- removed net INT: IC2.PD2(INT0), IC3.INT
- removed net MISO: IC2.PB4(MISO), IC3.SO, ISP1.MISO
- removed net MOSI: IC2.PB3(MOSI/OC2), IC3.SI, ISP1.MOSI
- removed net N$5: LSP1.MP, RN1C.1, RN1D.1
- removed net N$6: LSP2.MP, RN1A.1, RN1B.1
- removed net PC0: IC2.PC0(ADC0), R3.1
- removed net PC1: IC2.PC1(ADC1), R2.1
- removed net RELAIS_1: Q3.C, SV1.6
- removed net RELAIS_2: Q4.C, SV1.5
- removed net RST: IC2.PC6(/RESET), ISP1.RST, R1.1
- removed net SCK: IC2.PB5(SCK), IC3.SCK, ISP1.SCK
- removed net XTAL1: C3.2, IC2.PB6(XTAL1/TOSC1), Q1.1
- removed net XTAL2: C4.1, IC2.PB7(XTAL2/TOSC2), Q1.3
- removed net XTAL3: C5.2, IC3.OSC2, Q2.1
- removed net XTAL4: C6.1, IC3.OSC1, Q2.3
- new net +3,3V: JP2.1, X1.3V3A
- new net GPIO.06: IC1.INT, X1.GPIO06, X2.7
- new net MCP_VCC: C1.1, C3.1, IC1.VDD, IC2.VIO, JP2.2, R1.2
- new net N$4: C5.1, IC1.OSC2, Q1.1
- new net SPI_CE0: IC1.CS, X1.SPI_CE0, X2.3
- new net SPI_MISO: IC1.SO, X1.SPI_MISO, X2.4
- new net SPI_MOSI: IC1.SI, X1.SPI_MOSI, X2.5
- new net SPI_SCLK: IC1.SCK, X1.SPI_SCLK, X2.6
- net +24V: now also J1.4, J1.5, X3.2; no longer C1.1, IC1G$1.IN, SV1.4
- net +5V: now also IC2.VDD, JP2.3, X1.5V0A, X2.2; no longer C7.1, C8.1, C9.1, IC1G$1.OUT, IC2.AVCC, IC2.VCC@1, IC2.VCC@2, IC3.VDD, ISP1.VCC, R1.2, R4.2, RN1B.2, RN1C.2, U1.VDD, U1.VIO
- net CANH: now also IC2.CANH, J1.2, J1.7, JP1.1, X3.3; no longer SV1.2, U1.CANH
- net CANL: now also IC2.CANL, J1.1, J1.8, R2.1, X3.4; no longer SV1.1, U1.CANL
- net GND: now also C3.2, C5.2, IC1.VSS, IC2.STBY, IC2.VSS, J1.3, J1.6, J1.S1, J1.S2, X1.GND_A, X2.1, X3.1; no longer C10.2, C11.2, C3.1, C5.1, C6.2, C7.2, C8.2, C9.2, IC1G$1.GND, IC2.GND, IC2.GND@1, IC2.GND@2, IC3.VSS, ISP1.GND, Q1.2, Q1.4, Q2.2, Q2.4, Q3.E, Q4.E, SV1.3, U1.STBY, U1.VSS
- net N$1: now also C4.1, IC1.OSC1, Q1.2; no longer IC3.RESET, R4.1
- net N$2: now also IC1.RESET, R1.1; no longer Q3.B, R2.2
- net N$3: now also JP1.2, R2.2; no longer Q4.B, R3.2
- net RXCAN: now also IC1.RXCAN, IC2.RXD; no longer IC3.RXCAN, U1.RXD
- net TXCAN: now also IC1.TXCAN, IC2.TXD; no longer IC3.TXCAN, U1.TXD
Other:
- note added: "CAN-Shield MCP2515 / MCP 2562"
- note added: "Raspberry Pi"
- moved on the sheet: C1, C2, C3, C4, C5, R1, R2
