File: Backplane-4.brd (EAGLE design)
At the start: 194.3 x 84 mm, 12 parts, among them X1 FAC64SNO_DRILL, X2 FAC64SNO_DRILL, X3 FAC64SNO_DRILL, X4 FAC64SNO_DRILL, X5 FAC64SNO_DRILL, X6 FAC64SNO_DRILL, X7 FAC64SNO_DRILL, X8 FAC64SNO_DRILL

Commit message: Layouts angepasst
Parts:
- removed X5, X6, X7, X8: FAC64SNO_DRILL, my-con-vg:FAC64S_NO_DRILL
- moved SV2 96.5 mm to (92.1, 44.5)
- moved U$1 94.0 mm to (69.8, 57.1)
- moved U$2 94.0 mm to (69.8, 27.3)
- moved X4 5.08 mm to (82.5, 41.9)
Connections:
- net !PI_RESET: no longer X5.A26, X6.A26, X7.A26, X8.A26
- net +24V: no longer X5.A32, X5.C32, X6.A32, X6.C32, X7.A32, X7.C32, X8.A32, X8.C32
- net +3,3V: no longer X5.A2, X5.C2, X6.A2, X6.C2, X7.A2, X7.C2, X8.A2, X8.C2
- net +5V_EXT: no longer X5.A31, X5.C31, X6.A31, X6.C31, X7.A31, X7.C31, X8.A31, X8.C31
- net +5V_INT: no longer X5.A1, X5.C1, X6.A1, X6.C1, X7.A1, X7.C1, X8.A1, X8.C1
- net +5V_INT2: no longer X5.A28, X5.C28, X6.A28, X6.C28, X7.A28, X7.C28, X8.A28, X8.C28
- net 1WIRE: no longer X5.A7, X5.C7, X6.A7, X6.C7, X7.A7, X7.C7, X8.A7, X8.C7
- net A14: no longer X5.A14, X6.A14, X7.A14, X8.A14
- net A15: no longer X5.A15, X6.A15, X7.A15, X8.A15
- net A16: no longer X5.A16, X6.A16, X7.A16, X8.A16
- net A17: no longer X5.A17, X6.A17, X7.A17, X8.A17
- net A18: no longer X5.A18, X6.A18, X7.A18, X8.A18
- net A19: no longer X5.A19, X6.A19, X7.A19, X8.A19
- net A20: no longer X5.A20, X6.A20, X7.A20, X8.A20
- net A21: no longer X5.A21, X6.A21, X7.A21, X8.A21
- net A22: no longer X5.A22, X6.A22, X7.A22, X8.A22
- net A23: no longer X5.A23, X6.A23, X7.A23, X8.A23
- net A24: no longer X5.A24, X6.A24, X7.A24, X8.A24
- net A25: no longer X5.A25, X6.A25, X7.A25, X8.A25
- net GND: no longer X5.A11, X5.A13, X5.A27, X5.A29, X5.A3, X5.A6, X5.A8, X5.C13, X5.C29, X5.C3, X5.C6, X5.C8, X6.A11, X6.A13, X6.A27, X6.A29, X6.A3, X6.A6, X6.A8, X6.C13, X6.C29, X6.C3, X6.C6, X6.C8, X7.A11, X7.A13, X7.A27, X7.A29, X7.A3, X7.A6, X7.A8, X7.C13, X7.C29, X7.C3, X7.C6, X7.C8, X8.A11, X8.A13, X8.A27, X8.A29, X8.A3, X8.A6, X8.A8, X8.C13, X8.C29, X8.C3, X8.C6, X8.C8
- net GND_EXT: no longer X5.A30, X5.C30, X6.A30, X6.C30, X7.A30, X7.C30, X8.A30, X8.C30
- net GPIO.05: no longer X5.C14, X6.C14, X7.C14, X8.C14
- net GPIO.06: no longer X5.C15, X6.C15, X7.C15, X8.C15
- net GPIO.12: no longer X5.C16, X6.C16, X7.C16, X8.C16
- net GPIO.13: no longer X5.C17, X6.C17, X7.C17, X8.C17
- net GPIO.16: no longer X5.C18, X6.C18, X7.C18, X8.C18
- net GPIO.17: no longer X5.C19, X6.C19, X7.C19, X8.C19
- net GPIO.18: no longer X5.C20, X6.C20, X7.C20, X8.C20
- net GPIO.19: no longer X5.C21, X6.C21, X7.C21, X8.C21
- net GPIO.20: no longer X5.C22, X6.C22, X7.C22, X8.C22
- net GPIO.21: no longer X5.C23, X6.C23, X7.C23, X8.C23
- net GPIO.22: no longer X5.C24, X6.C24, X7.C24, X8.C24
- net GPIO.23: no longer X5.C25, X6.C25, X7.C25, X8.C25
- net GPIO.24: no longer X5.C26, X6.C26, X7.C26, X8.C26
- net GPIO.25: no longer X5.C27, X6.C27, X7.C27, X8.C27
- net I2C_SCL: no longer X5.A5, X5.C5, X6.A5, X6.C5, X7.A5, X7.C5, X8.A5, X8.C5
- net I2C_SDA: no longer X5.A4, X5.C4, X6.A4, X6.C4, X7.A4, X7.C4, X8.A4, X8.C4
- net PI_RXD: no longer X5.C12, X6.C12, X7.C12, X8.C12
- net PI_TXD: no longer X5.A12, X6.A12, X7.A12, X8.A12
- net SPI_CE0: no longer X5.A10, X6.A10, X7.A10, X8.A10
- net SPI_CE1: no longer X5.C11, X6.C11, X7.C11, X8.C11
- net SPI_MISO: no longer X5.A9, X6.A9, X7.A9, X8.A9
- net SPI_MOSI: no longer X5.C9, X6.C9, X7.C9, X8.C9
- net SPI_SCLK: no longer X5.C10, X6.C10, X7.C10, X8.C10
Routing:
- net +24V: track 369.6 -> 176.5 mm
- net +5V_INT: track 205.1 -> 88.3 mm
- net +3,3V: track 200.0 -> 88.3 mm
- net GPIO.25: track 194.3 -> 93.5 mm
- net GPIO.21: track 194.3 -> 93.5 mm
- net GPIO.12: track 194.3 -> 93.5 mm
- net GPIO.06: track 194.3 -> 93.5 mm
- net GPIO.05: track 194.3 -> 93.5 mm
- net GPIO.24: track 194.3 -> 93.5 mm
- net GPIO.23: track 194.3 -> 93.5 mm
- net GPIO.22: track 194.3 -> 93.5 mm
- net GPIO.20: track 194.3 -> 93.5 mm
- net GPIO.19: track 194.3 -> 93.5 mm
- net SPI_MOSI: track 194.3 -> 93.5 mm
- net PI_RXD: track 194.3 -> 93.5 mm
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Other:
- board size 194.3 x 84 mm -> 97.8 x 84 mm

Commit message: Verbesserte Stromversorgung, Pi-Kühler, CAN-Bus 8x-Schalter
Connections:
- removed net A24: SV1.47, SV2.47, X1.A24, X2.A24, X3.A24, X4.A24
- removed net A25: SV1.49, SV2.49, X1.A25, X2.A25, X3.A25, X4.A25
- new net +12V: SV1.47, SV1.49, SV2.47, SV2.49, X1.A24, X1.A25, X2.A24, X2.A25, X3.A24, X3.A25, X4.A24, X4.A25
Routing:
- net +12V: track 0.00 -> 174.8 mm
- net A25: track 87.4 -> 0.00 mm
- net A24: track 87.4 -> 0.00 mm
Changed lines of the file:
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@@
 <wire x1="87.63" y1="25.4" x2="90.805" y2="25.4" width="0.4064" layer="1"/>
 </signal>
-<signal name="A24">
+<signal name="+12V">
 <contactref element="X1" pad="A24"/>
 <contactref element="X2" pad="A24"/>
@@
 <wire x1="13.97" y1="22.86" x2="7.62" y2="22.86" width="0.4064" layer="1"/>
 <wire x1="87.63" y1="22.86" x2="90.805" y2="22.86" width="0.4064" layer="1"/>
-</signal>
-<signal name="A25">
 <contactref element="X1" pad="A25"/>
 <contactref element="X2" pad="A25"/>
@@
 <wire x1="13.97" y1="20.32" x2="7.62" y2="20.32" width="0.4064" layer="1"/>
 <wire x1="87.63" y1="20.32" x2="90.805" y2="20.32" width="0.4064" layer="1"/>
+<wire x1="87.63" y1="20.32" x2="86.36" y2="21.59" width="0" layer="19" extent="1-1"/>
 </signal>
 <signal name="TOP">
