File: CanBus-Gartensteuerung.brd (EAGLE design)
At the start: 100 x 100 mm, 90 parts, among them IC1 LM2937IMP-5.0, IC2 ATMEGA1284P, IC3 MCP2515T-I/SO, IC4 MCP2562-E/SN, IC5 ULN2003AD, IC6 ULN2003AD, IC7 PCF8574T, IC8 PCF8574T, IC9 PCF8574T, K1 HJR-4102-L, K10 HJR-4102-L, K11 36.11, K12 36.11, K2 HJR-4102-L, K3 HJR-4102-L, K4 HJR-4102-L, K5 HJR-4102-L, K6 HJR-4102-L, K7 HJR-4102-L, K8 HJR-4102-L, K9 HJR-4102-L, Q1 16MHz, Q2 16MHz, X1 22-27-2021-02, X10 22-27-2081-08, X11 22-27-2031-03, X12 22-27-2041-04, X13 22-27-2031-03, X14 22-27-2031-03, X2 22-27-2051-05, X3 22-27-2061-06, X4 22-27-2021-02, X5 22-27-2021-02, X6 MKDSN1,5/3-5,08, X7 MKDSN1,5/3-5,08, X8 22-27-2081-08, X9 22-27-2081-08

Commit message: Schaltpläne optimiert
Parts:
- added R20, R21: 10k, rcl:R0805
Connections:
- net +5V: now also R20.2, R21.2
- net CS: now also R20.1
- net INT_MCP: now also R21.1
Routing:
- net CS: track 19.0 -> 29.5 mm
- net +5V: track 275.3 -> 280.0 mm, vias 6 -> 7
- net INT_MCP: track 16.6 -> 20.3 mm
Other:
- board text added: "CAN-Bus Gartensteuerung Rev 2021/01 (c) Peter Müller"
- board text removed: "CAN-Bus Gartensteuerung Rev 2020/05 (c) Peter Müller"
Changed lines of the file:
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@@
 <setting verticaltext="up"/>
 </settings>
-<grid distance="1.27" unitdist="mm" unit="mm" style="lines" multiple="1" display="no" altdistance="12.5" altunitdist="mil" altunit="mil"/>
+<grid distance="1.27" unitdist="mm" unit="mm" style="dots" multiple="1" display="yes" altdistance="12.5" altunitdist="mil" altunit="mil"/>
 <layers>
 <layer number="1" name="Top" color="4" fill="1" visible="yes" active="yes"/>
@@
 <text x="56.515" y="66.3575" size="1.27" layer="21" font="vector" ratio="15" align="center">CAN-Bus
 Gartensteuerung
-Rev 2020/05
+Rev 2021/01
 (c) Peter Müller</text>
 <wire x1="14.2875" y1="62.23" x2="14.605" y2="62.23" width="0.254" layer="25"/>
@@
 </element>
 <element name="C7" library="rcl" package="C0805" value="100nF" x="27.94" y="56.515" smashed="yes" rot="R270">
-<attribute name="NAME" x="26.9875" y="57.4675" size="0.8128" layer="25" font="vector" align="center-right"/>
+<attribute name="NAME" x="26.9875" y="58.1025" size="0.8128" layer="25" font="vector" align="bottom-right"/>
 <attribute name="VALUE" x="25.4" y="57.785" size="1.27" layer="27" rot="R270"/>
 </element>
@@
 <attribute name="NAME" x="14.3144" y="91.4766" size="0.8128" layer="25" font="vector" align="top-left"/>
 <attribute name="VALUE" x="13.9969" y="90.3336" size="0.8128" layer="27" ratio="10"/>
+</element>
+<element name="R20" library="rcl" package="R0805" value="10k" x="27.6225" y="55.88" smashed="yes" rot="MR90">
+<attribute name="NAME" x="27.305" y="53.6575" size="0.8128" layer="26" font="vector" rot="MR0" align="top-center"/>
+<attribute name="VALUE" x="25.0825" y="55.245" size="1.27" layer="28" rot="MR90"/>
+</element>
+<element name="R21" library="rcl" package="R0805" value="10k" x="29.845" y="55.88" smashed="yes" rot="MR90">
+<attribute name="NAME" x="29.845" y="53.6575" size="0.8128" layer="26" font="vector" rot="MR0" align="top-center"/>
+<attribute name="VALUE" x="27.305" y="55.245" size="1.27" layer="28" rot="MR90"/>
 </element>
 </elements>
@@
 <contactref element="C9" pad="2"/>
 <wire x1="32.3" y1="68.11" x2="37.7825" y2="68.11" width="0.4064" layer="1"/>
-<wire x1="37.7825" y1="68.11" x2="37.7825" y2="66.675" width="0.4064" layer="1"/>
+<wire x1="37.7825" y1="68.11" x2="37.7825" y2="66.51" width="0.4064" layer="1"/>
 <wire x1="37.7825" y1="66.51" x2="37.7825" y2="62.865" width="0.4064" layer="1"/>
 <wire x1="37.7825" y1="62.865" x2="38.1" y2="62.5475" width="0.4064" layer="1"/>
@@
 <wire x1="38.89" y1="77.47" x2="39.3675" y2="76.9925" width="0.4064" layer="1"/>
 <wire x1="39.3675" y1="76.9925" x2="39.3675" y2="75.8825" width="0.4064" layer="1"/>
-<wire x1="27.94" y1="57.465" x2="22.2275" y2="57.465" width="0.4064" layer="1"/>
 <wire x1="18.4175" y1="61.275" x2="12.7" y2="61.275" width="0.4064" layer="1"/>
 <wire x1="12.7" y1="61.275" x2="2.54" y2="61.275" width="0.4064" layer="1"/>
@@
 <wire x1="37.7825" y1="68.11" x2="38.9" y2="69.2275" width="0.4064" layer="1"/>
 <wire x1="38.9" y1="69.2275" x2="38.9" y2="73.11" width="0.4064" layer="1"/>
-<wire x1="37.7825" y1="66.51" x2="37.7825" y2="66.675" width="0.4064" layer="1"/>
+<contactref element="R20" pad="2"/>
+<contactref element="R21" pad="2"/>
+<wire x1="29.845" y1="56.83" x2="27.6225" y2="56.83" width="0.3048" layer="16"/>
+<wire x1="22.23" y1="57.4675" x2="22.2275" y2="57.465" width="0.3048" layer="1"/>
+<wire x1="22.23" y1="57.4675" x2="25.4" y2="57.4675" width="0.3048" layer="1"/>
+<wire x1="25.4" y1="57.4675" x2="27.9375" y2="57.4675" width="0.3048" layer="1"/>
+<wire x1="27.9375" y1="57.4675" x2="27.94" y2="57.465" width="0.3048" layer="1"/>
+<wire x1="27.6225" y1="56.83" x2="26.0375" y2="56.83" width="0.3048" layer="16"/>
+<wire x1="26.0375" y1="56.83" x2="25.4" y2="57.4675" width="0.3048" layer="16"/>
+<via x="25.4" y="57.4675" extent="1-16" drill="0.35" diameter="0.7"/>
 </signal>
 <signal name="CANL">
@@
 <wire x1="32.0675" y1="58.7375" x2="32.7025" y2="59.3725" width="0.3048" layer="16"/>
 <wire x1="32.7025" y1="59.3725" x2="32.7025" y2="67.6275" width="0.3048" layer="16"/>
+<contactref element="R20" pad="1"/>
+<wire x1="32.385" y1="57.4675" x2="32.385" y2="53.0225" width="0.3048" layer="16"/>
+<wire x1="32.385" y1="53.0225" x2="31.75" y2="52.3875" width="0.3048" layer="16"/>
+<wire x1="27.6225" y1="54.93" x2="27.6225" y2="54.9275" width="0.3048" layer="16"/>
+<wire x1="27.6225" y1="54.9275" x2="30.1625" y2="52.3875" width="0.3048" layer="16"/>
+<wire x1="30.1625" y1="52.3875" x2="31.75" y2="52.3875" width="0.3048" layer="16"/>
 </signal>
 <signal name="XTAL1">
@@
 <wire x1="37.465" y1="55.7022" x2="37.465" y2="53.975" width="0.3048" layer="1"/>
 <wire x1="37.465" y1="53.975" x2="36.83" y2="53.34" width="0.3048" layer="1"/>
-<wire x1="36.83" y1="53.34" x2="34.925" y2="53.34" width="0.3048" layer="1"/>
-<via x="34.925" y="53.34" extent="1-16" drill="0.35" diameter="0.7"/>
-<wire x1="34.925" y1="53.34" x2="31.4325" y2="56.8325" width="0.3048" layer="16"/>
-<wire x1="31.4325" y1="56.8325" x2="31.4325" y2="59.055" width="0.3048" layer="16"/>
+<wire x1="36.83" y1="53.34" x2="31.4325" y2="53.34" width="0.3048" layer="1"/>
+<via x="31.4325" y="53.34" extent="1-16" drill="0.35" diameter="0.7"/>
+<wire x1="31.4325" y1="53.34" x2="31.4325" y2="54.9275" width="0.3048" layer="16"/>
+<wire x1="31.4325" y1="54.9275" x2="31.4325" y2="59.055" width="0.3048" layer="16"/>
 <wire x1="31.4325" y1="59.055" x2="31.75" y2="59.3725" width="0.3048" layer="16"/>
 <wire x1="31.75" y1="59.3725" x2="31.75" y2="62.23" width="0.3048" layer="16"/>
@@
 <wire x1="31.75" y1="62.23" x2="31.75" y2="63.31" width="0.3048" layer="1"/>
 <wire x1="31.75" y1="63.31" x2="32.3" y2="63.31" width="0.3048" layer="1"/>
+<contactref element="R21" pad="1"/>
+<wire x1="29.845" y1="54.93" x2="31.43" y2="54.93" width="0.3048" layer="16"/>
+<wire x1="31.43" y1="54.93" x2="31.4325" y2="54.9275" width="0.3048" layer="16"/>
 </signal>
 <signal name="INT_PCF">
@@
 <wire x1="45.72" y1="94.9325" x2="45.72" y2="94.2975" width="0.4064" layer="1"/>
 </signal>
+<signal name="N$3">
+</signal>
 </signals>
