File: CanBus-Gartensteuerung.sch (EAGLE design)
At the start: 89 parts, among them IC1 LM2937IMP-5.0, IC2 ATMEGA1284P, IC3 MCP2515T-I/SO, IC4 MCP2562-E/SN, IC5 ULN2003AD, IC6 ULN2003AD, IC7 PCF8574T, IC8 PCF8574T, IC9 PCF8574T, K1 HJR-4102-L, K10 HJR-4102-L, K11 36.11, K12 36.11, K2 HJR-4102-L, K3 HJR-4102-L, K4 HJR-4102-L, K5 HJR-4102-L, K6 HJR-4102-L, K7 HJR-4102-L, K8 HJR-4102-L, K9 HJR-4102-L, Q1 16MHz, Q2 16MHz, X1 22-27-2021-02, X10 22-27-2081-08, X11 22-27-2031-03, X12 22-27-2041-04, X13 22-27-2031-03, X14 22-27-2031-03, X2 22-27-2051-05, X3 22-27-2061-06, X4 22-27-2021-02, X5 22-27-2021-02, X6 MKDSN1,5/3-5,08, X7 MKDSN1,5/3-5,08, X8 22-27-2081-08, X9 22-27-2081-08

Commit message: Schaltpläne optimiert
Parts:
- added R20, R21: 10k, rcl:R-EU_R0805
Connections:
- net +5V: now also R20.2, R21.2
- net CS: now also R20.1
- net INT_MCP: now also R21.1
Other:
- note added: "0x46"
- note added: "CAN-Bus Gartensteuerung Rev. 2021/01 (c) Peter Müller <peter@crycode.de> https://crycode.de"
