File: Spannungsversorgung-3.sch (EAGLE design)
At the start: 28 parts, among them IC1 TI-INA226, U1 TSR2-2450, U2 TSR1-2433, U3 TSR1-2450, U4 TSR1-24120, X1 Ein/Aus, X2 MAC64L, X3 Eingang

Commit message: Schaltpläne optimiert
Other:
- note added: "HomePi - Spannungsversorgung Rev. 2020/04 (c) Peter Müller <peter@crycode.de> https://crycode.de"
- note removed: "HomePi - Spannungsversorgung Rev. 2019/05"
- moved on the sheet: A0, A1, C1, C2, C5, D1, F1, LED1, LED2, LED3, LED4, LED5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
